File: hardware/esp32v3_corebase/esp32v3_corebase.sch (KiCad schematic (older format))
At the start: 25 parts

Commit message: [FEATURE] Added CH340C with USB type C connector
Parts:
- removed U?: ESP32, QFN48-0.4MM, symbol SparkFun-RF:ESP32
- added C14: 10nF, Capacitors:0603, symbol Device:C_Small
- added D1, D2: LED, LED_SMD:LED_0603_1608Metric, symbol Device:LED
- added J1: USB_C_Receptacle_USB2.0, Connector_USB:USB_C_Receptacle_Palconn_UTC16-G, symbol Connector:USB_C_Receptacle_USB2.0
- added Q1: MBT2222ADW1T1, Package_TO_SOT_SMD:SOT-363_SC-70-6, symbol Transistor_BJT:MBT2222ADW1T1
- added R1, R11, R12: 10kR, Resistors:0603, symbol Device:R_US
- added R10, R9: 5k1R, Resistors:0603, symbol Device:R_US
- added R13, R14: 560R, Resistors:0603, symbol Device:R_US
- added U4: CH340C, Package_SO:SOIC-16_3.9x9.9mm_P1.27mm, symbol Interface_USB:CH340G
- added U5: ESP32, Package_DFN_QFN:QFN-48-1EP_6x6mm_P0.4mm_EP4.2x4.2mm, symbol SparkFun-RF:ESP32
- C1, C10, C11, C12, C13, C15, C2, C3, C4, C5, C6, C7, C8, C9: renamed from C?; footprint (none) -> Capacitors:0603
- R2, R3, R4, R5, R6, R7, R8: renamed from R?; footprint (none) -> Resistors:0603
- U1: renamed from U?; symbol Regulator_Linear:TLV75533PDBV -> esp32v3_corebase-rescue:TLV75533PDBV-Regulator_Linear
- U3: renamed from U?; footprint SOIC-8 -> Silicon-Standard:SOIC-8
- Y1: renamed from Y?; footprint (none) -> Clocks:CRYSTAL-SMD-3.2X2.5MM
Connections:
- net +3V3: now also R13.2, R14.2, U4.16 (VCC), U5.1 (VDDA), U5.19 (VDD3P3_RTC), U5.3 (VDDA3P3), U5.37 (VDD3P3_CPU), U5.4 (VDDA3P3), U5.43 (VDDA), U5.46 (VDDA)
- net ANT: now also U5.2 (LNA_IN)
- net BOOT: now also Q1.4 (E2), U5.23 ((ADC2:1/TOUCH1/RTC11/CLK_OUT1)GPIO0)
- net GND: now also C14.2, J1.A1 (GND), J1.A12 (GND), J1.B1 (GND), J1.B12 (GND), J1.S1 (SHIELD), R10.2, R9.2, U4.1 (GND), U5.47 (CAP2), U5.49 (EP_GND)
- net GPIO12: now also U5.18 ((GPIO12/ADC2:5/TOUCH5/RTC15/SPIQ)MTDI)
- net GPIO15: now also U5.21 ((GPIO15/ADC2:3/TOUCH3/RTC13/SPICSO/U0RTS)MTDO)
- net GPIO2: now also U5.22 ((ADC2:2/TOUCH2/RTC12/SPIWP)GPIO2)
- net GPIO32: now also U5.12 (32K_XP(GPIO32/ADC1:4/TOUCH9/RTC9))
- net GPIO33: now also U5.13 (32K_XN(GPIO33/ADC1:5/TOUCH8/RTC8))
- net RESET: now also Q1.6 (C1), U5.9 (CHIP_PU)
- net SD_CS: now also U5.30 ((GPIO11/SPICSO/HS1_CMD/U1RTS)SD_CMD)
- net SD_D0: now also U5.32 ((GPIO7/SPI1/HS1_DATA0)SD_DATA0)
- net SD_D1: now also U5.33 ((GPIO8/SPID/HS1_DATA1)SD_DATA1)
- net SD_D2: now also U5.28 ((GPIO9/SPIHD/HS1_DATA2/U1RX)SD_DATA2)
- net SD_D3: now also U5.29 ((GPIO10/SPIWP/HS1_DATA3/U1TX)SD_DATA3)
- net SD_SCK: now also U5.31 ((GPIO6/SPICLK/HS1_CLK/U1CTS)SD_CLK)
- net SD_SDIO: now also U5.26 (VDD3P3_SDIO)
- net URX: now also D1.1 (K), U4.2 (TXD), U5.40 ((GPIO3/CLK_OUT2/HS2_DATA0)U0RXD)
- net UTX: now also D2.1 (K), U4.3 (RXD)
- net VIN: now also R1.2
- net at R8.2: now also U5.41 ((GPIO1/CLK_OUT3/HS2_DATA1)U0TXD)
- net at C3.1, Y1.3: now also U5.44 (XTAL_N)
- net at C2.1, Y1.1: now also U5.45 (XTAL_P)
- net at C9.1, R2.1: now also U5.48 (CAP1)
- net LDO_EN: no longer names the net of U1.3 (EN)
- net LDO_EN: now also R1.1
- new net: C14.1, U4.4 (V3)
- new net: J1.A5 (CC1), R9.1
- new net: J1.B5 (CC2), R10.1
- new net: Q1.2 (B1), R11.1
- new net: Q1.5 (B2), R12.1
- new net: D1.2 (A), R13.1
- new net: D2.2 (A), R14.1
- new net COM_CTS: Q1.1 (E1), R12.2, U4.9 (~CTS)
- new net COM_DTR: Q1.3 (C2), R11.2, U4.13 (~DTR)
- new net D+: J1.A6 (D+), J1.B6 (D+), U4.5 (UD+)
- new net D-: J1.A7 (D-), J1.B7 (D-), U4.6 (UD-)
- new net GPIO13: U5.20 ((GPIO13/ADC2:4/TOUCH4/RTC14/SPID/U0CTS)MTCK)
- new net GPIO14: U5.17 ((GPIO14/ADC2:6/TOUCH6/RTC16/SPICLK)MTMS)
- new net GPIO16: U5.25 ((HS1_DATA4)GPIO16)
- new net GPIO17: U5.27 ((HS1_DATA5)GPIO17)
- new net GPIO18: U5.35 ((VSPICLK/HS1_DATA7)GPIO18)
- new net GPIO19: U5.38 ((VSPIQ/HS2_DATA2)GPIO19)
- new net GPIO21: U5.42 ((VSPIHD/HS2_CMD)GPIO21)
- new net GPIO22: U5.39 ((VSPIWP/HS2_CLK)GPIO22)
- new net GPIO23: U5.36 (GPIO23)
- new net GPIO25: U5.14 ((DAC1/ADC2:8/RTC6)GPIO25)
- new net GPIO26: U5.15 ((DAC2/ADC2:9/RTC7)GPIO26)
- new net GPIO27: U5.16 ((ADC2:7/TOUCH7/RTC17)GPIO27)
- new net GPIO34: U5.10 (VDET_1(GPI34/ADC1:6))
- new net GPIO35: U5.11 (VDET_2(GPI35/ADC1:7))
- new net GPIO36: U5.5 (SENSOR_VP(GPI36/ADC1:0/RTC0))
- new net GPIO37: U5.6 (SENSOR_CAPP(GPI37/ADC1:1/RTC1))
- new net GPIO38: U5.7 (SENSOR_CAPN(GPI38/ADC1:2/RTC2))
- new net GPIO39: U5.8 (SENSOR_VN(GPI39/ADC1:3/RTC3))
- new net GPIO4: U5.24 ((ADC2:0/TOUCH0/RTC10/SPIHD)GPIO4)
- new net GPIO5: U5.34 ((VSPICS0/HS1_DATA6)GPIO5)
- new net VBUS: J1.A4 (VBUS), J1.A9 (VBUS), J1.B4 (VBUS), J1.B9 (VBUS)
- no-connect marks 0 -> 9
Other:
- moved on the sheet: C10, C2, C3, C5, C6, C7, C8, C9, R2, R8, Y1

Commit message: [FEATURE] Changed resistors and capacitors footprint from 0603 to 0402
Parts:
- C1, C12, C13, C14, C15, C5: footprint Capacitors:0603 -> Capacitor_SMD:C_0603_1608Metric
- C10, C11, C2, C3, C4, C6, C7, C8, C9: footprint Capacitors:0603 -> Capacitor_SMD:C_0402_1005Metric
- R1, R10, R11, R12, R2, R3, R4, R5, R6, R7, R8, R9: footprint Resistors:0603 -> Resistor_SMD:R_0402_1005Metric
- R13, R14: footprint Resistors:0603 -> Resistor_SMD:R_0603_1608Metric
Changed lines of the file:
@@
 F 0 "C1" H 900 6950 50  0000 L CNN
 F 1 "1uF" H 900 6750 50  0000 L CNN
-F 2 "Capacitors:0603" H 850 6850 50  0001 C CNN
+F 2 "Capacitor_SMD:C_0603_1608Metric" H 850 6850 50  0001 C CNN
 F 3 "~" H 850 6850 50  0001 C CNN
 	1    850  6850
@@
 F 0 "C4" H 1200 6950 50  0000 L CNN
 F 1 "100nF" H 1200 6750 50  0000 L CNN
-F 2 "Capacitors:0603" H 1150 6850 50  0001 C CNN
+F 2 "Capacitor_SMD:C_0402_1005Metric" H 1150 6850 50  0001 C CNN
 F 3 "~" H 1150 6850 50  0001 C CNN
 	1    1150 6850
@@
 F 0 "C11" H 2600 6950 50  0000 L CNN
 F 1 "100nF" H 2600 6750 50  0000 L CNN
-F 2 "Capacitors:0603" H 2550 6850 50  0001 C CNN
+F 2 "Capacitor_SMD:C_0402_1005Metric" H 2550 6850 50  0001 C CNN
 F 3 "~" H 2550 6850 50  0001 C CNN
 	1    2550 6850
@@
 F 0 "C12" H 2900 6950 50  0000 L CNN
 F 1 "1uF" H 2900 6750 50  0000 L CNN
-F 2 "Capacitors:0603" H 2850 6850 50  0001 C CNN
+F 2 "Capacitor_SMD:C_0603_1608Metric" H 2850 6850 50  0001 C CNN
 F 3 "~" H 2850 6850 50  0001 C CNN
 	1    2850 6850
@@
 F 0 "C13" H 3250 6950 50  0000 L CNN
 F 1 "10uF" H 3250 6750 50  0000 L CNN
-F 2 "Capacitors:0603" H 3200 6850 50  0001 C CNN
+F 2 "Capacitor_SMD:C_0603_1608Metric" H 3200 6850 50  0001 C CNN
 F 3 "~" H 3200 6850 50  0001 C CNN
 	1    3200 6850
@@
 F 0 "R5" V 4950 6550 50  0000 C CNN
 F 1 "10kR" V 4950 6800 50  0000 C CNN
-F 2 "Resistors:0603" V 5090 6690 50  0001 C CNN
+F 2 "Resistor_SMD:R_0402_1005Metric" V 5090 6690 50  0001 C CNN
 F 3 "~" H 5050 6700 50  0001 C CNN
 	1    5050 6700
@@
 F 0 "R6" V 4950 6750 50  0000 C CNN
 F 1 "10kR" V 4950 7000 50  0000 C CNN
-F 2 "Resistors:0603" V 5090 6890 50  0001 C CNN
+F 2 "Resistor_SMD:R_0402_1005Metric" V 5090 6890 50  0001 C CNN
 F 3 "~" H 5050 6900 50  0001 C CNN
 	1    5050 6900
@@
 F 0 "R7" V 4950 6950 50  0000 C CNN
 F 1 "10kR" V 4950 7200 50  0000 C CNN
-F 2 "Resistors:0603" V 5090 7090 50  0001 C CNN
+F 2 "Resistor_SMD:R_0402_1005Metric" V 5090 7090 50  0001 C CNN
 F 3 "~" H 5050 7100 50  0001 C CNN
 	1    5050 7100
@@
 F 0 "R4" V 4050 6750 50  0000 C CNN
 F 1 "10kR" V 4050 7000 50  0000 C CNN
-F 2 "Resistors:0603" V 4190 6890 50  0001 C CNN
+F 2 "Resistor_SMD:R_0402_1005Metric" V 4190 6890 50  0001 C CNN
 F 3 "~" H 4150 6900 50  0001 C CNN
 	1    4150 6900
@@
 F 0 "R3" V 4050 6550 50  0000 C CNN
 F 1 "10kR" V 4050 6800 50  0000 C CNN
-F 2 "Resistors:0603" V 4190 6690 50  0001 C CNN
+F 2 "Resistor_SMD:R_0402_1005Metric" V 4190 6690 50  0001 C CNN
 F 3 "~" H 4150 6700 50  0001 C CNN
 	1    4150 6700
@@
 F 0 "C15" H 10450 1250 50  0000 L CNN
 F 1 "1uF" H 10400 1150 50  0000 L CNN
-F 2 "Capacitors:0603" H 10350 1250 50  0001 C CNN
+F 2 "Capacitor_SMD:C_0603_1608Metric" H 10350 1250 50  0001 C CNN
 F 3 "~" H 10350 1250 50  0001 C CNN
 	1    10350 1250
@@
 F 0 "R11" V 9500 2200 50  0000 C CNN
 F 1 "10kR" V 9700 2200 50  0000 C CNN
-F 2 "Resistors:0603" V 9640 2190 50  0001 C CNN
+F 2 "Resistor_SMD:R_0402_1005Metric" V 9640 2190 50  0001 C CNN
 F 3 "~" H 9600 2200 50  0001 C CNN
 	1    9600 2200
@@
 F 0 "R12" V 9500 2850 50  0000 C CNN
 F 1 "10kR" V 9700 2850 50  0000 C CNN
-F 2 "Resistors:0603" V 9640 2840 50  0001 C CNN
+F 2 "Resistor_SMD:R_0402_1005Metric" V 9640 2840 50  0001 C CNN
 F 3 "~" H 9600 2850 50  0001 C CNN
 	1    9600 2850
@@
 F 0 "C9" H 2250 4000 50  0000 L CNN
 F 1 "3.3nF" H 2250 3800 50  0000 L CNN
-F 2 "Capacitors:0603" H 2200 3900 50  0001 C CNN
+F 2 "Capacitor_SMD:C_0402_1005Metric" H 2200 3900 50  0001 C CNN
 F 3 "~" H 2200 3900 50  0001 C CNN
 	1    2200 3900
@@
 F 0 "C7" H 1750 4000 50  0000 L CNN
 F 1 "10nF" H 1750 3800 50  0000 L CNN
-F 2 "Capacitors:0603" H 1700 3900 50  0001 C CNN
+F 2 "Capacitor_SMD:C_0402_1005Metric" H 1700 3900 50  0001 C CNN
 F 3 "~" H 1700 3900 50  0001 C CNN
 	1    1700 3900
@@
 F 0 "R2" V 1850 3550 50  0000 C CNN
 F 1 "20kR" V 1850 3800 50  0000 C CNN
-F 2 "Resistors:0603" V 1990 3690 50  0001 C CNN
+F 2 "Resistor_SMD:R_0402_1005Metric" V 1990 3690 50  0001 C CNN
 F 3 "~" H 1950 3700 50  0001 C CNN
 	1    1950 3700
@@
 F 0 "R8" V 6795 1000 50  0000 C CNN
 F 1 "R_US" V 6886 1000 50  0000 C CNN
-F 2 "Resistors:0603" V 7040 990 50  0001 C CNN
+F 2 "Resistor_SMD:R_0402_1005Metric" V 7040 990 50  0001 C CNN
 F 3 "~" H 7000 1000 50  0001 C CNN
 	1    7000 1000
@@
 F 0 "C3" V 1150 2250 50  0000 L CNN
 F 1 "10pF" V 1150 2450 50  0000 L CNN
-F 2 "Capacitors:0603" H 1100 2400 50  0001 C CNN
+F 2 "Capacitor_SMD:C_0402_1005Metric" H 1100 2400 50  0001 C CNN
 F 3 "~" H 1100 2400 50  0001 C CNN
 	1    1100 2400
@@
 F 0 "C2" V 1150 1750 50  0000 L CNN
 F 1 "10pF" V 1150 1950 50  0000 L CNN
-F 2 "Capacitors:0603" H 1100 1900 50  0001 C CNN
+F 2 "Capacitor_SMD:C_0402_1005Metric" H 1100 1900 50  0001 C CNN
 F 3 "~" H 1100 1900 50  0001 C CNN
 	1    1100 1900
@@
 F 0 "C10" H 2400 1250 50  0000 L CNN
 F 1 "100nF" H 2400 1050 50  0000 L CNN
-F 2 "Capacitors:0603" H 2350 1150 50  0001 C CNN
+F 2 "Capacitor_SMD:C_0402_1005Metric" H 2350 1150 50  0001 C CNN
 F 3 "~" H 2350 1150 50  0001 C CNN
 	1    2350 1150
@@
 F 0 "C8" H 2050 1250 50  0000 L CNN
 F 1 "100nF" H 2050 1050 50  0000 L CNN
-F 2 "Capacitors:0603" H 2000 1150 50  0001 C CNN
+F 2 "Capacitor_SMD:C_0402_1005Metric" H 2000 1150 50  0001 C CNN
 F 3 "~" H 2000 1150 50  0001 C CNN
 	1    2000 1150
@@
 F 0 "C6" H 1700 1250 50  0000 L CNN
 F 1 "100nF" H 1700 1050 50  0000 L CNN
-F 2 "Capacitors:0603" H 1650 1150 50  0001 C CNN
+F 2 "Capacitor_SMD:C_0402_1005Metric" H 1650 1150 50  0001 C CNN
 F 3 "~" H 1650 1150 50  0001 C CNN
 	1    1650 1150
@@
 F 0 "C5" H 1350 1250 50  0000 L CNN
 F 1 "1uF" H 1350 1050 50  0000 L CNN
-F 2 "Capacitors:0603" H 1300 1150 50  0001 C CNN
+F 2 "Capacitor_SMD:C_0603_1608Metric" H 1300 1150 50  0001 C CNN
 F 3 "~" H 1300 1150 50  0001 C CNN
 	1    1300 1150
@@
 F 0 "R9" H 9050 4650 50  0000 C CNN
 F 1 "5k1R" V 9050 4800 50  0000 C CNN
-F 2 "Resistors:0603" V 8990 4740 50  0001 C CNN
+F 2 "Resistor_SMD:R_0402_1005Metric" V 8990 4740 50  0001 C CNN
 F 3 "~" H 8950 4750 50  0001 C CNN
 	1    8950 4750
@@
 F 0 "R10" H 9050 4650 50  0000 C CNN
 F 1 "5k1R" V 9050 4800 50  0000 C CNN
-F 2 "Resistors:0603" V 9190 4740 50  0001 C CNN
+F 2 "Resistor_SMD:R_0402_1005Metric" V 9190 4740 50  0001 C CNN
 F 3 "~" H 9150 4750 50  0001 C CNN
 	1    9150 4750
@@
 F 0 "C14" H 9500 4600 50  0000 L CNN
 F 1 "10nF" H 9500 4400 50  0000 L CNN
-F 2 "Capacitors:0603" H 9450 4500 50  0001 C CNN
+F 2 "Capacitor_SMD:C_0603_1608Metric" H 9450 4500 50  0001 C CNN
 F 3 "~" H 9450 4500 50  0001 C CNN
 	1    9450 4500
@@
 F 0 "R1" H 1600 7050 50  0000 C CNN
 F 1 "10kR" H 1600 7150 50  0000 C CNN
-F 2 "Resistors:0603" V 1540 6940 50  0001 C CNN
+F 2 "Resistor_SMD:R_0402_1005Metric" V 1540 6940 50  0001 C CNN
 F 3 "~" H 1500 6950 50  0001 C CNN
 	1    1500 6950
@@
 F 0 "R14" H 10600 4150 50  0000 C CNN
 F 1 "560R" V 10600 4300 50  0000 C CNN
-F 2 "Resistors:0603" V 10740 4240 50  0001 C CNN
+F 2 "Resistor_SMD:R_0603_1608Metric" V 10740 4240 50  0001 C CNN
 F 3 "~" H 10700 4250 50  0001 C CNN
 	1    10700 4250
@@
 F 0 "R13" H 10600 4150 50  0000 C CNN
 F 1 "560R" V 10600 4300 50  0000 C CNN
-F 2 "Resistors:0603" V 10540 4240 50  0001 C CNN
+F 2 "Resistor_SMD:R_0603_1608Metric" V 10540 4240 50  0001 C CNN
 F 3 "~" H 10500 4250 50  0001 C CNN
 	1    10500 4250

Commit message: [FEATURE] Minor changes on the circuit and VIN to 5V
Parts:
- added C?: 10uF, Capacitor_SMD:C_0402_1005Metric, symbol Device:C_Small
- added C?: 10nF, Capacitor_SMD:C_0402_1005Metric, symbol Device:C_Small
- added C?: 22uF, Capacitor_SMD:C_0402_1005Metric, symbol Device:C_Small
- added D?: B230A, symbol Device:D_Schottky
- added F?: Polyfuse_Small, symbol Device:Polyfuse_Small
- added L?: 6.8uH, symbol Device:L_Small
- added R?: 62k, Resistor_SMD:R_0402_1005Metric, symbol Device:R_US
- added R?: 11k8, Resistor_SMD:R_0402_1005Metric, symbol Device:R_US
- added U?: RT8259GE, Package_TO_SOT_SMD:SOT-23-6, symbol Buck_Regulators:RT8259GE
Connections:
- net GND: now also C?.2, C?.2, D?.2 (A), R?.1, U?.2 (GND)
- net VBUS: now also F?.1; no longer J1.A4 (VBUS), J1.A9 (VBUS), J1.B4 (VBUS), J1.B9 (VBUS)
- net VIN renamed +5V
- net +5V: now also C?.1, L?.2, R?.2
- new net: F?.2, J1.A4 (VBUS), J1.A9 (VBUS), J1.B4 (VBUS), J1.B9 (VBUS)
- new net: C?.1, U?.1 (BOOT)
- new net: C?.2, D?.1 (K), L?.1, U?.6 (PHASE)
- new net: R?.1, R?.2, U?.~ (FB)
- new net PD_IN: C?.1, U?.5 (VIN)
- no-connect marks 9 -> 10
Other:
- note added: "4.7uH and 19k6R for 3.33V output\n6.8uH and 11k8R for 5V output"
- note added: "BAT54 or 1N4148"
- note added: "Bootloader Circuit"
- note added: "Buck Converter for PD with 1.2A"
- note added: "USB to Serial Interface"
- note added: "VOUT = 0.8(1+(R1/R2))"
- moved on the sheet: C1, C11, C12, C13, C14, C15, C4, D1, D2, J1, Q1A, Q1B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
